File: Hardware/SparkFun_GPS_ZED-F9R_BoB.brd (EAGLE design)
At the start: 43.2 x 50.8 mm, 140 parts, among them J1 U.FL, J3 QWIIC_RIGHT_ANGLE, J4 QWIIC_RIGHT_ANGLE, U1 DUAL-OPTO_HCPL-073L, U2 U-BLOX_ZED_F9R, U3 UHS_INVERTER_SCHMITT_TRIGGERS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, U4 UHS_INVERTER_SCHMITT_TRIGGERS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, U5 3.3V

Commit message: Replaces silk with coool skull
Parts:
- U$19: device Dead#Reckoning#GPS#board#silk#FINAL#png:DEAD#RECKONING#GPS#BOARD#SILK#FINAL#PNG -> Dead#Reckoning#GPS#board#silk#FINAL#png:DEAD#RECKONING#GPS#BOARD#SILK#FINAL#JPG
- U$20: device Dead#Reckoning#GPS#board#silk#FINALSMALL:DEAD#RECKONING#GPS#BOARD#SILK#FINAL#PNG -> Dead#Reckoning#GPS#board#silk#FINALSMALL:DEAD#RECKONING#GPS#BOARD#SILK#FINAL#JPG
- moved U$20 1.40 mm to (6.35, 11.4)
- moved U$19 0.85 mm to (22.9, 22.9)
Changed lines of the file:
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@@
 <layer number="27" name="tValues" color="7" fill="1" visible="no" active="yes"/>
 <layer number="28" name="bValues" color="7" fill="1" visible="no" active="yes"/>
-<layer number="29" name="tStop" color="7" fill="3" visible="yes" active="yes"/>
+<layer number="29" name="tStop" color="7" fill="3" visible="no" active="yes"/>
 <layer number="30" name="bStop" color="7" fill="6" visible="no" active="yes"/>
 <layer number="31" name="tCream" color="7" fill="4" visible="no" active="yes"/>
@@
 <layer number="37" name="tTest" color="7" fill="1" visible="no" active="yes"/>
 <layer number="38" name="bTest" color="7" fill="1" visible="no" active="yes"/>
-<layer number="39" name="tKeepout" color="4" fill="11" visible="yes" active="yes"/>
+<layer number="39" name="tKeepout" color="4" fill="11" visible="no" active="yes"/>
 <layer number="40" name="bKeepout" color="1" fill="11" visible="no" active="yes"/>
 <layer number="41" name="tRestrict" color="4" fill="10" visible="no" active="yes"/>
@@
 <layer number="115" name="ReferenceISLANDS" color="7" fill="1" visible="no" active="no"/>
 <layer number="116" name="Patch_BOT" color="9" fill="4" visible="no" active="no"/>
-<layer number="117" name="PM_Ref" color="26" fill="1" visible="yes" active="yes"/>
+<layer number="117" name="PM_Ref" color="26" fill="1" visible="no" active="yes"/>
 <layer number="118" name="Rect_Pads" color="7" fill="1" visible="no" active="no"/>
-<layer number="119" name="PF_Ref" color="31" fill="1" visible="yes" active="yes"/>
-<layer number="120" name="WFL_Ref" color="25" fill="1" visible="yes" active="yes"/>
+<layer number="119" name="PF_Ref" color="31" fill="1" visible="no" active="yes"/>
+<layer number="120" name="WFL_Ref" color="25" fill="1" visible="no" active="yes"/>
 <layer number="121" name="_tsilk" color="7" fill="1" visible="no" active="no"/>
 <layer number="122" name="_bsilk" color="7" fill="1" visible="no" active="no"/>
@@
 <attribute name="PROD_ID" value="RES-15081" x="35.433" y="22.225" size="1.778" layer="27" rot="R270" display="off"/>
 </element>
-<element name="U$19" library="Dead#Reckoning#GPS#board#silk#FINAL#png" package="DEAD#RECKONING#GPS#BOARD#SILK#FINAL#PNG" value="" x="22.098" y="22.479" smashed="yes" rot="MR0"/>
-<element name="U$20" library="Dead#Reckoning#GPS#board#silk#FINALSMALL" package="DEAD#RECKONING#GPS#BOARD#SILK#FINAL#PNG" value="" x="7.747" y="11.43" smashed="yes"/>
 <element name="U$25" library="dead reckoning" package="GPS_DEAD_RECKONING0" value="" x="32.004" y="33.274" smashed="yes" rot="MR0"/>
+<element name="U$19" library="Dead#Reckoning#GPS#board#silk#FINAL#png" package="DEAD#RECKONING#GPS#BOARD#SILK#FINAL#JPG" value="" x="22.86" y="22.86" smashed="yes" rot="MR0"/>
+<element name="U$20" library="Dead#Reckoning#GPS#board#silk#FINALSMALL" package="DEAD#RECKONING#GPS#BOARD#SILK#FINAL#JPG" value="" x="6.35" y="11.43" smashed="yes"/>
 </elements>
 <signals>
