File: Hardware/SparkFun_ZED-F9R_v12_uFL.sch (EAGLE design)
At the start: 77 parts, among them J1 U.FL, J3 QWIIC_RIGHT_ANGLE, J4 QWIIC_RIGHT_ANGLE, U1 DUAL-OPTO_HCPL-073LSOIC-8, U3 UHS_INVERTER_SCHMITT_TRIGGERS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, U4 UHS_INVERTER_SCHMITT_TRIGGERS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, U5 3.3V, U6 U-BLOX_ZED-F9R

Commit message: Removes older files, adds new measures and ordering instructions
Parts:
- added LOGO5: SPECIAL_INSTRUCTIONS-ORDERING, SparkFun-Aesthetics:SPECIAL_INSTRUCTIONS-ORDERING
Other:
- note added: "GNSS/Dead Reckoning Module - u-blox ZED-F9R"
- note removed: "GNSS/Dead Reckoning Module - ublox ZED-F9R"
Changed lines of the file:
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@@
 <part name="GND27" library="SparkFun-PowerSymbols" deviceset="GND" device=""/>
 <part name="J1" library="SparkFun-Connectors" deviceset="U.FL" device="" value="U.FL"/>
+<part name="LOGO5" library="SparkFun-Aesthetics" deviceset="SPECIAL_INSTRUCTIONS" device="-ORDERING"/>
 </parts>
 <sheets>
@@
 <text x="421.64" y="7.62" size="2.54" layer="94" font="vector">v12</text>
 <text x="349.25" y="11.43" size="2.54" layer="94" font="vector">Elias Santistevan</text>
-<text x="86.36" y="269.24" size="2.54" layer="94" font="vector" align="center">GNSS/Dead Reckoning Module - ublox ZED-F9R</text>
+<text x="86.36" y="269.24" size="2.54" layer="94" font="vector" align="center">GNSS/Dead Reckoning Module - u-blox ZED-F9R</text>
 <text x="388.112" y="272.034" size="2.54" layer="94" font="vector" align="center">Battery - MS421R</text>
 <text x="355.6" y="127" size="2.54" layer="94" font="vector" align="center">Connectors</text>
@@
 <attribute name="NAME" x="161.29" y="80.264" size="1.778" layer="95"/>
 </instance>
+<instance part="LOGO5" gate="G$1" x="386.08" y="30.48" smashed="yes"/>
 </instances>
 <busses>
