File: Production/SparkFun_GPS_ZED-F9R_BoB-Panel.brd (EAGLE design)
At the start: 100.6 x 129.8 mm, 581 parts, among them J1 U.FL, J12 QWIIC_RIGHT_ANGLE, J15 QWIIC_RIGHT_ANGLE, J16 U.FL, J19 QWIIC_RIGHT_ANGLE, J22 QWIIC_RIGHT_ANGLE, J23 U.FL, J26 QWIIC_RIGHT_ANGLE, J3 QWIIC_RIGHT_ANGLE, J4 QWIIC_RIGHT_ANGLE, J8 QWIIC_RIGHT_ANGLE, J9 U.FL, U1 DUAL-OPTO_HCPL-073L, U10 UHS_INVERTER_SCHMITT_TRIGGERS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, U11 3.3V, U12 U-BLOX_ZED_F9R, U13 DUAL-OPTO_HCPL-073L, U14 UHS_INVERTER_SCHMITT_TRIGGERS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, U15 UHS_INVERTER_SCHMITT_TRIGGERS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, U16 3.3V, U17 U-BLOX_ZED_F9R, U18 DUAL-OPTO_HCPL-073L, U19 UHS_INVERTER_SCHMITT_TRIGGERS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, U2 U-BLOX_ZED_F9R, U20 UHS_INVERTER_SCHMITT_TRIGGERS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, U3 UHS_INVERTER_SCHMITT_TRIGGERS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, U4 UHS_INVERTER_SCHMITT_TRIGGERS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, U5 3.3V, U6 3.3V, U7 U-BLOX_ZED_F9R, U8 DUAL-OPTO_HCPL-073L, U9 UHS_INVERTER_SCHMITT_TRIGGERS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

Commit message: Fixes silk and repanelizes
Parts:
- U$110, U$181, U$252: device wt_dir:D#0 -> SparkFun-Aesthetics:SFE_LOGO_FLAME_.2
- U$111, U$182, U$253: device wt_dir:D#1 -> Labels:SCL-[)
- U$112, U$183, U$254: device wt_dir:W#2 -> Labels:SDA-[)
- U$113, U$184, U$255: device wt_dir:W#3 -> Labels:3V3-04
- U$114, U$185, U$256: device SparkFun-Aesthetics:SFE_LOGO_FLAME_.2 -> Labels:GND-04
- U$115, U$186, U$257: device Labels:SCL-[) -> Labels:3V3-04
- U$116, U$187, U$258: device Labels:SDA-[) -> Labels:GND-04
- U$117, U$188, U$259: device Labels:3V3-04 -> Labels:MISO-(]-04
- U$118, U$189, U$260: device Labels:GND-04 -> Labels:MOSI-(]-04
- U$119, U$190, U$261: device Labels:3V3-04 -> wt_dir:D#0
- U$120, U$191, U$262: device Labels:GND-04 -> wt_dir:D#1
- U$121, U$192, U$263: device Labels:MISO-(]-04 -> wt_dir:W#2
- U$122, U$193, U$264: device Labels:MOSI-(]-04 -> wt_dir:W#3
- U$123, U$194, U$265: device wt_dir:D#0 -> Labels:5V
- U$124, U$195, U$266: device wt_dir:D#1 -> ALL_LABELS:INT1
- U$125, U$196, U$267: device wt_dir:W#2 -> ALL_LABELS:PPS4
- U$126, U$197, U$268: device wt_dir:W#3 -> Labels:GND-04
- U$127, U$198, U$269: device Labels:5V -> moar:TXO21
- U$128, U$199, U$270: device ALL_LABELS:INT1 -> txr_rxi:RXI22
- U$129, U$200, U$271: device ALL_LABELS:PPS4 -> txr_rxi:SCLK1
- U$130, U$201, U$272: device Labels:GND-04 -> txr_rxi:TXR0
- U$131, U$202, U$273: device moar:TXO21 -> dead reckoning:GPS_DEAD_RECKONING0
- U$132, U$203, U$274: device txr_rxi:RXI22 -> Dead#Reckoning#GPS#board#silk#FINAL#png:DEAD#RECKONING#GPS#BOARD#SILK#FINAL#JPG
- U$133, U$204, U$275: device txr_rxi:SCLK1 -> Dead#Reckoning#GPS#board#silk#FINALSMALL:DEAD#RECKONING#GPS#BOARD#SILK#FINAL#JPG
- U$134, U$205, U$276: device txr_rxi:TXR0 -> Orientation:X1
- U$135, U$206, U$277: device dead reckoning:GPS_DEAD_RECKONING0 -> Orientation:Y2
- U$136, U$207, U$278: device Dead#Reckoning#GPS#board#silk#FINAL#png:DEAD#RECKONING#GPS#BOARD#SILK#FINAL#JPG -> Orientation:Y2
- U$137, U$208, U$279: device Dead#Reckoning#GPS#board#silk#FINALSMALL:DEAD#RECKONING#GPS#BOARD#SILK#FINAL#JPG -> Orientation:Z0
- U$138, U$209, U$280: device Orientation:X1 -> Orientation:Z0
- U$139, U$210, U$281: device Orientation:Y2 -> D+,D-:D#0
- U$140, U$211, U$282: device Orientation:Y2 -> D+,D-:W#2
- U$141, U$212, U$283: device Orientation:Z0 -> D+,D-:D#1
- U$142, U$213, U$284: device Orientation:Z0 -> D+,D-:W#3
- U$60: device wt_dir:D#0 -> D+,D-:D#0
- U$61: device wt_dir:D#1 -> D+,D-:W#2
- U$64: device wt_dir:W#2 -> D+,D-:D#1
- U$65: device wt_dir:W#3 -> D+,D-:W#3
- moved U$113 41.5 mm to (45.3, 34.3), flipped to the top, turned to 0 degrees
- moved U$255 41.5 mm to (45.3, 88.1), flipped to the top, turned to 0 degrees
- moved U$184 41.5 mm to (1.65, 88.1), flipped to the top, turned to 0 degrees
- moved U$112 41.4 mm to (45.3, 31.8), flipped to the top, turned to 0 degrees
- moved U$183 41.4 mm to (1.65, 85.6), flipped to the top, turned to 0 degrees
- moved U$254 41.4 mm to (45.3, 85.6), flipped to the top, turned to 0 degrees
- moved U$111 38.7 mm to (45.3, 29.2), flipped to the top, turned to 0 degrees
- moved U$253 38.7 mm to (45.3, 83.0), flipped to the top, turned to 0 degrees
- moved U$182 38.7 mm to (1.65, 83.0), flipped to the top, turned to 0 degrees
- moved U$201 37.2 mm to (1.57, 80.4), turned to 0 degrees
- moved U$272 37.2 mm to (45.3, 80.4), turned to 0 degrees
- moved U$130 37.2 mm to (45.3, 26.6), turned to 0 degrees
- moved U$124 36.7 mm to (45.3, 19.1)
- moved U$266 36.7 mm to (45.3, 72.9)
- moved U$195 36.7 mm to (1.57, 72.9)
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