File: Production/SparkFun_ZED-F9R_v11-Panel.brd (EAGLE design)
At the start: 43.2 x 50.8 mm, 154 parts, among them J3 QWIIC_RIGHT_ANGLE, J4 QWIIC_RIGHT_ANGLE, U1 DUAL-OPTO_HCPL-073LSOIC-8, U3 UHS_INVERTER_SCHMITT_TRIGGERS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, U4 UHS_INVERTER_SCHMITT_TRIGGERS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, U5 3.3V, U6 U-BLOX_ZED-F9R

Commit message: Adds new Production files and a few vias to the board design
Parts:
- removed FRAME1: FRAME-LEDGER, SparkFun-Aesthetics:CREATIVE_COMMONS
- added $1_25_$_2020-03-30_22-52-01, $1_25_$_2020-03-30_22-52-02, $1_25_$_2020-03-30_22-52-03, H10, H11, H12, H3, H5, H6, H7, H8, H9: STAND-OFFTIGHT, SparkFun-Hardware:STAND-OFF-TIGHT
- added BT1, BT3, BT4: RELOWABLE_BATTERY_MS421R, SparkFun-Batteries:MS421R_IV03E
- added C13, C25, C37: 47pF, SparkFun-Capacitors:0402
- added C14, C15, C16, C26, C27, C28, C38, C39, C40: 1.0uF, SparkFun-Capacitors:0402-TIGHT
- added C17, C18, C29, C30, C41, C42: 1nF, SparkFun-Capacitors:0402
- added C19, C20, C21, C22, C24, C31, C32, C33, C34, C36, C43, C44, C45, C46, C48: 0.1uF, SparkFun-Capacitors:0402-TIGHT
- added C23, C35, C47: 2.2uF, SparkFun-Capacitors:0402-TIGHT
- added D10, D19, D28: 0.5A/40V/420mV, SparkFun-DiscreteSemi:SOD-323
- added D11, D20, D29: RED, SparkFun-LED:LED-0603
- added D12, D21, D30: PRTR5V0U2F, SparkFun-IC-Power:SOT886
- added D13, D14, D15, D22, D23, D24, D31, D32, D33: BLUE, SparkFun-LED:LED-0603
- added D16, D17, D25, D26, D34, D35: 15V, SparkFun-DiscreteSemi:SOT23-3
- added D18, D27, D36: PESD0402-0402, SparkFun-DiscreteSemi:0402
- added E$1, E$2, E$3, E$4: (no value), SparkFun-Aesthetics:FIDUCIAL-1X2
- added E$5, E$6: (no value), SparkFun-Retired:FIDUCIAL-1.5X3
- added E2, E3, E4: ANTENNA-SMA-GROUNDEDEDGE_SMA, SparkFun-RF:SMA-EDGE
- added FB2, FB3, FB4: 120Ω, SparkFun-Coils:0402
- added FD10, FD11, FD12, FD13, FD14, FD15, FD16, FD5, FD6, FD7, FD8, FD9: FIDUCIALUFIDUCIAL, SparkFun-Aesthetics:FIDUCIAL-MICRO
- added GEO1, GEO2, GEO3, PPS1, PPS2, PPS3, PWR1, PWR2, PWR3, RTK1, RTK2, RTK3, SHIELD1, SHIELD2, SHIELD3: JUMPER-SMT_2_NC_TRACE_SILK, SparkFun-Jumpers:SMT-JUMPER_2_NC_TRACE_SILK
- added I2C1, I2C2, I2C3: JUMPER-SMT_3_2-NC_TRACE_SILK, SparkFun-Jumpers:SMT-JUMPER_3_2-NC_TRACE_SILK
- added J1, J10, J13, J16, J19, J22: QWIIC_RIGHT_ANGLE, SparkFun-Connectors:JST04_1MM_RA
- added J11, J17, J23: (no value), SparkFun-Connectors:1X06_NO_SILK
- added J12, J18, J24: (no value), SparkFun-Connectors:1X09_NO_SILK
- added J14, J20, J8: (no value), SparkFun-Connectors:1X11_NO_SILK
- added J15, J21, J9: (no value), SparkFun-Connectors:USB-C-16P-2LAYER-PADS
- added LOGO10, LOGO12, LOGO14, LOGO16, LOGO6, LOGO8: QWIIC_LOGO_4MM, SparkFun-Aesthetics:QWIIC_4MM
- added LOGO11, LOGO15, LOGO7: OSHW-LOGOS, SparkFun-Aesthetics:OSHW-LOGO-S
- added LOGO13, LOGO5, LOGO9: SFE_LOGO_NAME_FLAME.2_INCH, SparkFun-Aesthetics:SFE_LOGO_NAME_FLAME_.2
- added R25, R26, R49, R50, R73, R74: 2.2K, SparkFun-Resistors:0402
- added R27, R39, R41, R51, R63, R65, R75, R87, R89: 3.3k, SparkFun-Resistors:0603
- added R28, R52, R76: 1KOHM-0402-1/16W-1%, SparkFun-Resistors:0402
- added R29, R30, R53, R54, R77, R78: 5.1k, SparkFun-Resistors:0402
- added R31, R32, R55, R56, R79, R80: 27, SparkFun-Resistors:0603
- added R33, R34, R38, R57, R58, R62, R81, R82, R86: 2.2k, SparkFun-Resistors:0603
- added R35, R37, R59, R61, R83, R85: 33, SparkFun-Resistors:0603
- added R36, R60, R84: 100K, SparkFun-Resistors:0402
- added R40, R42, R64, R66, R88, R90: 470, SparkFun-Resistors:0603
- added R43, R44, R67, R68, R91, R92: 910, SparkFun-Resistors:0603
- added R45, R46, R47, R48, R69, R70, R71, R72, R93, R94, R95, R96: 33, SparkFun-Resistors:1206_RA
- added SPI1, SPI2, SPI3: JUMPER-SMT_2_NO_SILK, SparkFun-Jumpers:SMT-JUMPER_2_NO_SILK
- added TP2, TP3, TP4: TEST-POINT3X5, SparkFun-Connectors:PAD.03X.05
- added U$100, U$174, U$248: (no value), top:#W##245
- added U$101, U$175, U$249: (no value), top:RXI229
- added U$102, U$141, U$176, U$215, U$250, U$289: (no value), top:BLK18
- added U$103, U$140, U$177, U$214, U$251, U$288: (no value), top:GRN19
- added U$104, U$178, U$252: (no value), top:PWR6
- added U$105, U$179, U$253: (no value), top:RTK12
- added U$106, U$180, U$254: (no value), top:GEO10
- added U$107, U$181, U$255: (no value), top:PPS8
- added U$108, U$182, U$256: (no value), top:ZED#F9R21
- added U$109, U$183, U$257: (no value), top:L1#L26
- added U$110, U$184, U$258: (no value), top:ANTENNA6
- added U$111, U$112, U$185, U$186, U$259, U$260: (no value), top:X17
- added U$113, U$114, U$187, U$188, U$261, U$262: (no value), top:Z19
- added U$115, U$116, U$189, U$190, U$263, U$264: (no value), top:Y18
- added U$117, U$191, U$265: (no value), top:TXO2234
- added U$118, U$192, U$266: (no value), top:##RST##28
- added U$119, U$193, U$267: (no value), top:##CS##25
- added U$120, U$194, U$268: (no value), top:##CS##26
- added U$121, U$195, U$269: (no value), top:#SCL#SCLK#2243
- added U$122, U$196, U$270: (no value), top:#D##2249
- added U$123, U$197, U$271: (no value), top:#D##2248
- added U$124, U$198, U$272: (no value), top:#W##2253
- added U$125, U$199, U$273: (no value), top:#W##2252
- added U$126, U$200, U$274: (no value), top:#TXR#2255
- added U$127, U$201, U$275: (no value), top:##RST##27
- added U$128, U$202, U$276: (no value), top:##SFBT##29
- added U$129, U$203, U$277: (no value), top:#PPS#2
- added U$130, U$204, U$278: (no value), top:#SCL#SCLK#2244
- added U$131, U$205, U$279: (no value), top:#GEO#12
- added U$132, U$206, U$280: (no value), top:#RTK#14
- added U$133, U$207, U$281: (no value), top:#PPS#10
- added U$134, U$208, U$282: (no value), top:#PWR#8
- added U$135, U$209, U$283: (no value), top:#I2C#5
- added U$136, U$210, U$284: (no value), top:#SPI#4
- added U$137, U$151, U$152, U$153, U$154, U$155, U$211, U$225, U$226, U$227, U$228, U$229, U$285, U$77, U$78, U$79, U$80, U$81: (no value), top:#GND#16
- added U$138, U$212, U$286: (no value), top:#RXI2#34
- added U$139, U$213, U$287: (no value), top:#TXO2#235
- added U$142, U$216, U$290: (no value), top:GPS_DEAD_RECKONING24
- added U$143, U$217, U$291: (no value), top:ZED#F9R25
- added U$144, U$218, U$292: (no value), top:#SHLD#2258
- added U$145, U$219, U$293: (no value), top:#INT#1
- added U$146, U$220, U$294: (no value), top:#INT#0
- added U$147, U$221, U$295: (no value), top:#RXI#CIPO#32
- added U$148, U$222, U$296: (no value), top:#TXO#COPI#33
- added U$149, U$223, U$75: (no value), Dead#Reckoning#GPS#board#silk#FINAL#png:DEAD#RECKONING#GPS#BOARD#SILK#FINAL#JPG
- added U$150, U$224, U$76: (no value), Dead#Reckoning#GPS#board#silk#FINALSMALL:DEAD#RECKONING#GPS#BOARD#SILK#FINAL#JPG
- added U$156, U$157, U$158, U$159, U$230, U$231, U$232, U$233, U$82, U$83, U$84, U$85: (no value), top:#3V3#17
- added U$160, U$161, U$234, U$235, U$86, U$87: (no value), top:#5V#17
- added U$162, U$236, U$88: (no value), top:#SDA#235
- added U$163, U$237, U$89: (no value), top:#SDA#236
- added U$164, U$238, U$90: (no value), top:#SCL#238
- added U$165, U$239, U$91: (no value), top:#TXR#248
- added U$166, U$240, U$92: (no value), top:##SFBT##26
- added U$167, U$241, U$93: (no value), top:#PPS#3
- added U$168, U$242, U$94: (no value), top:#COPI#230
- added U$169, U$243, U$95: (no value), top:#CIPO#232
- added U$170, U$244, U$96: (no value), top:#SCLK#233
- added U$171, U$245, U$97: (no value), top:#D##241
- added U$172, U$246, U$98: (no value), top:#D##240
- added U$173, U$247, U$99: (no value), top:#W##244
- added U10, U15, U20: U-BLOX_ZED-F9R, SparkFun-GPS:UBLOX_ZED_F9R
- added U11, U16, U2: 3.3V, SparkFun-IC-Power:SOT23-5
- added U12, U17, U7: DUAL-OPTO_HCPL-073LSOIC-8, SparkFun-DiscreteSemi:SO08
- added U13, U14, U18, U19, U8, U9: UHS_INVERTER_SCHMITT_TRIGGERSIP6, SparkFun-IC-Amplifiers:SIP6_MICROPAK2
Connections:
- new net !RESET1: J12.4, R46.P2
- new net !RESET2: J18.4, R70.P2
- new net !RESET3: J24.4, R94.P2
- new net !SAFEBOOT1: J12.3, R46.P3
- new net !SAFEBOOT2: J18.3, R70.P3
- new net !SAFEBOOT3: J24.3, R94.P3
- new net 3.3V1: C15.1, C16.1, C19.1, C20.1, C21.1, C22.1, C24.1, D10.A, D11.A, D14.A, I2C1.2, J1.2, J10.2, J12.8, J8.3, R36.2, R43.2, R44.2, U10.P33, U10.P34, U10.P38, U2.5, U7.8, U8.P6, U9.P6
- new net 3.3V2: C27.1, C28.1, C31.1, C32.1, C33.1, C34.1, C36.1, D19.A, D20.A, D23.A, I2C2.2, J13.2, J14.3, J16.2, J18.8, R60.2, R67.2, R68.2, U11.5, U12.8, U13.P6, U14.P6, U15.P33, U15.P34, U15.P38
- new net 3.3V3: C39.1, C40.1, C43.1, C44.1, C45.1, C46.1, C48.1, D28.A, D29.A, D32.A, I2C3.2, J19.2, J20.3, J22.2, J24.8, R84.2, R91.2, R92.2, U16.5, U17.8, U18.P6, U19.P6, U20.P33, U20.P34, U20.P38
- new net DIR+1: J8.9, R41.1
- new net DIR+2: J14.9, R65.1
- new net DIR+3: J20.9, R89.1
- new net DIR_IN1: R42.2, U7.4
- new net DIR_IN2: R66.2, U12.4
- new net DIR_IN3: R90.2, U17.4
- new net DIR_INV1: R44.1, U7.6, U9.P2
- new net DIR_INV2: R68.1, U12.6, U14.P2
- new net DIR_INV3: R92.1, U17.6, U19.P2
- new net DIR_OUT1: R47.P6, U9.P4
- new net DIR_OUT2: R71.P6, U14.P4
- new net DIR_OUT3: R95.P6, U19.P4
- new net DMINUS1: R31.2, U10.P39
- new net DMINUS2: R55.2, U15.P39
- new net DMINUS3: R79.2, U20.P39
- new net DPLUS1: R32.2, U10.P40
- new net DPLUS2: R56.2, U15.P40
- new net DPLUS3: R80.2, U20.P40
- new net D_SEL1: SPI1.1, U10.P47
- new net D_SEL2: SPI2.1, U15.P47
- new net D_SEL3: SPI3.1, U20.P47
- new net GEOF_STAT1: D15.A, R48.P7
- new net GEOF_STAT2: D24.A, R72.P7
- new net GEOF_STAT3: D33.A, R96.P7
- new net GND1: BT1.-, C13.2, C14.2, C15.2, C16.2, C17.2, C18.2, C19.2, C20.2, C21.2, C22.2, C23.2, C24.2, D12.2, D16.1, D17.1, D18.1, E2.GND@0, E2.GND@1, E2.GND@2, E2.GND@3, GEO1.1, J1.1, J10.1, J11.6, J12.9, J8.1, J8.10, J8.8, J9.GND, J9.GND2, PPS1.1, PWR1.1, R29.1, R30.1, R36.1, SHIELD1.1, SPI1.2, U10.G1, U10.G10, U10.G11, U10.G12, U10.G13, U10.G14, U10.G15, U10.G16, U10.G17, U10.G18, U10.G19, U10.G2, U10.G20, U10.G21, U10.G22, U10.G23, U10.G24, U10.G25, U10.G26, U10.G27, U10.G28, U10.G29, U10.G3, U10.G30, U10.G31, U10.G32, U10.G33, U10.G34, U10.G35, U10.G36, U10.G37, U10.G38, U10.G39, U10.G4, U10.G40, U10.G41, U10.G42, U10.G43, U10.G44, U10.G45, U10.G46, U10.G47, U10.G48, U10.G5, U10.G6, U10.G7, U10.G8, U10.G9, U10.P1, U10.P12, U10.P14, U10.P3, U10.P32, U10.P37, U10.P41, U10.P48, U2.2, U7.2, U7.3, U7.5, U8.P3, U9.P3
- new net GND2: BT3.-, C25.2, C26.2, C27.2, C28.2, C29.2, C30.2, C31.2, C32.2, C33.2, C34.2, C35.2, C36.2, D21.2, D25.1, D26.1, D27.1, E3.GND@0, E3.GND@1, E3.GND@2, E3.GND@3, GEO2.1, J13.1, J14.1, J14.10, J14.8, J15.GND, J15.GND2, J16.1, J17.6, J18.9, PPS2.1, PWR2.1, R53.1, R54.1, R60.1, SHIELD2.1, SPI2.2, U11.2, U12.2, U12.3, U12.5, U13.P3, U14.P3, U15.G1, U15.G10, U15.G11, U15.G12, U15.G13, U15.G14, U15.G15, U15.G16, U15.G17, U15.G18, U15.G19, U15.G2, U15.G20, U15.G21, U15.G22, U15.G23, U15.G24, U15.G25, U15.G26, U15.G27, U15.G28, U15.G29, U15.G3, U15.G30, U15.G31, U15.G32, U15.G33, U15.G34, U15.G35, U15.G36, U15.G37, U15.G38, U15.G39, U15.G4, U15.G40, U15.G41, U15.G42, U15.G43, U15.G44, U15.G45, U15.G46, U15.G47, U15.G48, U15.G5, U15.G6, U15.G7, U15.G8, U15.G9, U15.P1, U15.P12, U15.P14, U15.P3, U15.P32, U15.P37, U15.P41, U15.P48
- new net GND3: BT4.-, C37.2, C38.2, C39.2, C40.2, C41.2, C42.2, C43.2, C44.2, C45.2, C46.2, C47.2, C48.2, D30.2, D34.1, D35.1, D36.1, E4.GND@0, E4.GND@1, E4.GND@2, E4.GND@3, GEO3.1, J19.1, J20.1, J20.10, J20.8, J21.GND, J21.GND2, J22.1, J23.6, J24.9, PPS3.1, PWR3.1, R77.1, R78.1, R84.1, SHIELD3.1, SPI3.2, U16.2, U17.2, U17.3, U17.5, U18.P3, U19.P3, U20.G1, U20.G10, U20.G11, U20.G12, U20.G13, U20.G14, U20.G15, U20.G16, U20.G17, U20.G18, U20.G19, U20.G2, U20.G20, U20.G21, U20.G22, U20.G23, U20.G24, U20.G25, U20.G26, U20.G27, U20.G28, U20.G29, U20.G3, U20.G30, U20.G31, U20.G32, U20.G33, U20.G34, U20.G35, U20.G36, U20.G37, U20.G38, U20.G39, U20.G4, U20.G40, U20.G41, U20.G42, U20.G43, U20.G44, U20.G45, U20.G46, U20.G47, U20.G48, U20.G5, U20.G6, U20.G7, U20.G8, U20.G9, U20.P1, U20.P12, U20.P14, U20.P3, U20.P32, U20.P37, U20.P41, U20.P48
- new net INT1: J12.2, R46.P4
- new net INT2: J18.2, R70.P4
- new net INT3: J24.2, R94.P4
- new net N$100: R71.P4, U15.P22
- new net N$101: R71.P3, U15.P23
- new net N$102: GEO2.2, R62.1
- new net N$103: D24.C, R62.2
- new net N$104: C30.1, D25.3, R63.2, R64.1
- new net N$105: C29.1, D26.3, R65.2, R66.1
- new net N$106: D28.C, R75.2
- new net N$107: I2C3.1, R73.2
- new net N$108: I2C3.3, R74.2
- new net N$109: J21.B5, R77.2
- new net N$110: J21.A5, R78.2
- new net N$111: R82.1, RTK3.2
- new net N$112: PPS3.2, R81.1
- new net N$113: D31.C, R81.2
- new net N$114: D32.C, R82.2
- new net N$115: D29.C, R76.2
- new net N$116: PWR3.2, R76.1
- new net N$117: C37.1, FB4.2, R83.1
- new net N$118: D30.3, J21.A6, J21.B6
- new net N$119: D30.1, J21.A7, J21.B7
- new net N$120: D30.6, R79.1
- new net N$121: D30.4, R80.1
- new net N$122: R94.P7, U20.P49
- new net N$123: R94.P5, U20.P51
- new net N$124: R93.P6, U20.P44
- new net N$125: R93.P5, U20.P45
- new net N$126: R94.P8, U20.P46
- new net N$127: R93.P8, U20.P42
- new net N$128: R93.P7, U20.P43
- new net N$129: R95.P1, U20.P27
- new net N$13: D10.C, R27.2
- new net N$130: R95.P2, U20.P26
- new net N$131: R96.P2, U20.P19
- new net N$132: R96.P1, U20.P20
- new net N$133: R85.1, U20.P53
- new net N$134: R94.P6, U20.P50
- new net N$135: R95.P4, U20.P22
- new net N$136: R95.P3, U20.P23
- new net N$137: GEO3.2, R86.1
- new net N$138: D33.C, R86.2
- new net N$139: C42.1, D34.3, R87.2, R88.1
- new net N$140: C41.1, D35.3, R89.2, R90.1
- new net N$36: I2C1.1, R25.2
- new net N$38: I2C1.3, R26.2
- new net N$39: J9.B5, R29.2
- new net N$40: J9.A5, R30.2
- new net N$41: R34.1, RTK1.2
- new net N$42: PPS1.2, R33.1
- new net N$43: D13.C, R33.2
- new net N$44: D14.C, R34.2
- new net N$45: D11.C, R28.2
- new net N$46: PWR1.2, R28.1
- new net N$47: C13.1, FB2.2, R35.1
- new net N$48: D12.3, J9.A6, J9.B6
- new net N$49: D12.1, J9.A7, J9.B7
- new net N$50: D12.6, R31.1
- new net N$51: D12.4, R32.1
- new net N$52: R46.P7, U10.P49
- new net N$53: R46.P5, U10.P51
- new net N$54: R45.P6, U10.P44
- new net N$55: R45.P5, U10.P45
- new net N$56: R46.P8, U10.P46
- new net N$57: R45.P8, U10.P42
- new net N$58: R45.P7, U10.P43
- new net N$59: R47.P1, U10.P27
- new net N$60: R47.P2, U10.P26
- new net N$61: R48.P2, U10.P19
- new net N$62: R48.P1, U10.P20
- new net N$63: R37.1, U10.P53
- new net N$64: R46.P6, U10.P50
- new net N$65: R47.P4, U10.P22
- new net N$66: R47.P3, U10.P23
- new net N$67: GEO1.2, R38.1
- new net N$68: D15.C, R38.2
- new net N$69: C18.1, D16.3, R39.2, R40.1
- new net N$70: C17.1, D17.3, R41.2, R42.1
- new net N$71: D19.C, R51.2
- new net N$72: I2C2.1, R49.2
- new net N$73: I2C2.3, R50.2
- new net N$74: J15.B5, R53.2
- new net N$75: J15.A5, R54.2
- new net N$76: R58.1, RTK2.2
- new net N$77: PPS2.2, R57.1
- new net N$78: D22.C, R57.2
- new net N$79: D23.C, R58.2
- new net N$80: D20.C, R52.2
- new net N$81: PWR2.2, R52.1
- new net N$82: C25.1, FB3.2, R59.1
- new net N$83: D21.3, J15.A6, J15.B6
- new net N$84: D21.1, J15.A7, J15.B7
- new net N$85: D21.6, R55.1
- new net N$86: D21.4, R56.1
- new net N$87: R70.P7, U15.P49
- new net N$88: R70.P5, U15.P51
- new net N$89: R69.P6, U15.P44
- new net N$90: R69.P5, U15.P45
- new net N$91: R70.P8, U15.P46
- new net N$92: R69.P8, U15.P42
- new net N$93: R69.P7, U15.P43
- new net N$94: R71.P1, U15.P27
- new net N$95: R71.P2, U15.P26
- new net N$96: R72.P2, U15.P19
- new net N$97: R72.P1, U15.P20
- new net N$98: R61.1, U15.P53
- new net N$99: R70.P6, U15.P50
- new net PPS1: D13.A, J12.1, R37.2
- new net PPS2: D22.A, J18.1, R61.2
- new net PPS3: D31.A, J24.1, R85.2
- new net RF_IN1: D18.2, E2.SIG, FB2.1, U10.P2
- new net RF_IN2: D27.2, E3.SIG, FB3.1, U15.P2
- new net RF_IN3: D36.2, E4.SIG, FB4.1, U20.P2
- new net RTK_STAT1: R48.P8, RTK1.1
- new net RTK_STAT2: R72.P8, RTK2.1
- new net RTK_STAT3: R96.P8, RTK3.1
- new net RXI/CIPO1: J8.5, R45.P2
- new net RXI/CIPO2: J14.5, R69.P2
- new net RXI/CIPO3: J20.5, R93.P2
- new net RXI1: J11.3, R47.P7
- new net RXI3: J17.3, R71.P7
- new net RXI4: J23.3, R95.P7
- new net SCL/CLK1: J1.4, J10.4, J12.6, J8.7, R26.1, R45.P4
- new net SCL/CLK2: J13.4, J14.7, J16.4, J18.6, R50.1, R69.P4
- new net SCL/CLK3: J19.4, J20.7, J22.4, J24.6, R74.1, R93.P4
- new net SDA/!CS1: J1.3, J10.3, J12.7, J8.4, R25.1, R45.P3
- new net SDA/!CS2: J13.3, J14.4, J16.3, J18.7, R49.1, R69.P3
- new net SDA/!CS3: J19.3, J20.4, J22.3, J24.7, R73.1, R93.P3
- new net SHIELD1: J9.SHLD1, J9.SHLD2, J9.SHLD3, J9.SHLD4, SHIELD1.2
- new net SHIELD2: J15.SHLD1, J15.SHLD2, J15.SHLD3, J15.SHLD4, SHIELD2.2
- new net SHIELD3: J21.SHLD1, J21.SHLD2, J21.SHLD3, J21.SHLD4, SHIELD3.2
- new net TXO/COPI1: J8.6, R45.P1
- new net TXO/COPI2: J14.6, R69.P1
- new net TXO/COPI3: J20.6, R93.P1
- new net TXO1: J11.2, R47.P8
- new net TXO3: J17.2, R71.P8
- new net TXO4: J23.2, R95.P8
- new net TX_READY1: J12.5, R46.P1
- new net TX_READY2: J18.5, R70.P1
- new net TX_READY3: J24.5, R94.P1
- new net VIN1: C14.1, D12.5, J8.2, J9.VBUS1, J9.VBUS2, U2.1, U2.3
- new net VIN2: C26.1, D21.5, J14.2, J15.VBUS1, J15.VBUS2, U11.1, U11.3
- new net VIN3: C38.1, D30.5, J20.2, J21.VBUS1, J21.VBUS2, U16.1, U16.3
- new net V_BATT1: BT1.+, C23.1, R27.1, TP2.1, U10.P36
- new net V_BATT2: BT3.+, C35.1, R51.1, TP3.1, U15.P36
- new net V_BATT3: BT4.+, C47.1, R75.1, TP4.1, U20.P36
- new net V_RF1: R35.2, U10.P7
- new net V_RF2: R59.2, U15.P7
- new net V_RF3: R83.2, U20.P7
- new net WT+1: J8.11, R39.1
- new net WT+2: J14.11, R63.1
- new net WT+3: J20.11, R87.1
- new net WT_IN1: R40.2, U7.1
- new net WT_IN2: R64.2, U12.1
- new net WT_IN3: R88.2, U17.1
- new net WT_INV1: R43.1, U7.7, U8.P2
- new net WT_INV2: R67.1, U12.7, U13.P2
- new net WT_INV3: R91.1, U17.7, U18.P2
- new net WT_OUT1: R47.P5, U8.P4
- new net WT_OUT2: R71.P5, U13.P4
- new net WT_OUT3: R95.P5, U18.P4
Routing:
- net 3.3V2: track 0.00 -> 143.3 mm, vias 0 -> 13
- net 3.3V3: track 0.00 -> 143.3 mm, vias 0 -> 13
- net 3.3V1: track 0.00 -> 143.3 mm, vias 0 -> 13
- net SCL/CLK3: track 0.00 -> 95.8 mm, vias 0 -> 6
- net SCL/CLK2: track 0.00 -> 95.8 mm, vias 0 -> 6
- net SCL/CLK1: track 0.00 -> 95.8 mm, vias 0 -> 6
- net SDA/!CS2: track 0.00 -> 82.1 mm, vias 0 -> 5
- net SDA/!CS1: track 0.00 -> 82.1 mm, vias 0 -> 5
- net SDA/!CS3: track 0.00 -> 82.1 mm, vias 0 -> 5
- net VIN1: track 0.00 -> 51.1 mm, vias 0 -> 6
- net VIN3: track 0.00 -> 51.1 mm, vias 0 -> 6
- net VIN2: track 0.00 -> 51.1 mm, vias 0 -> 6
- net RXI/CIPO3: track 0.00 -> 50.8 mm, vias 0 -> 2
- net RXI/CIPO1: track 0.00 -> 50.8 mm, vias 0 -> 2
- net RXI/CIPO2: track 0.00 -> 50.8 mm, vias 0 -> 2
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- added copper zone on layer 1, net GND1
- added copper zone on layer 16, net GND1
- added copper zone on layer 1, net GND2
- added copper zone on layer 16, net GND2
- added copper zone on layer 1, net GND3
- added copper zone on layer 16, net GND3
- added copper zone on layer 1, net RF_IN1
- added copper zone on layer 1, net RF_IN2
- added copper zone on layer 1, net RF_IN3
- added copper zone on layer 1, net SHIELD1
- added copper zone on layer 16, net SHIELD1
- added copper zone on layer 1, net SHIELD2
- added copper zone on layer 16, net SHIELD2
- added copper zone on layer 1, net SHIELD3
- added copper zone on layer 16, net SHIELD3
Other:
- board size 43.2 x 50.8 mm -> 100.6 x 146.8 mm
- board text added: "Route Out"
- board text added: "v-score"
- board text removed: "Elias Santistevan"
- board text removed: "Units In Inches"
